Commit message: training update

File: robot.urdf (robot description, URDF)
Before this commit: robot C:\Users\daniel\Downloads\gradus-simulation, 4 links, 3 joints
Links:
- link arm_1: geometry collision mesh filename=package://assets/arm_1.stl; visual mesh filename=package://assets/arm_1.stl
- link arm_2: geometry collision mesh filename=package://assets/arm_2.stl; visual mesh filename=package://assets/arm_2.stl
- link beam_1: geometry collision mesh filename=package://assets/beam_1.stl; collision mesh filename=package://assets/beam_1.stl
- link holder: geometry collision mesh filename=package://assets/base.stl; collision mesh filename=package://assets/holder.stl

Commit message: reward function

File: robot.urdf (robot description, URDF)
Before this commit: robot gradus-simulation, 4 links, 3 joints
Joints:
- joint cart: limit lower=-0.28 upper=0.35 effort=10 velocity=10 -> lower=-0.38 upper=0.45 effort=10 velocity=10
